File: 1.hardware/motor_42/motor_42.kicad_pcb (KiCad board)
At the start: 2 copper layers, 40 x 40 mm, 5 parts, among them U1 STM32F103RBTx

Commit message: 중간 저장
Parts:
- added C28: 0.1uF/16V, Capacitor_SMD:C_0402_1005Metric, F.Cu at (109.9, 74.2)
- added C29: 0.1uF/16V, Capacitor_SMD:C_0402_1005Metric, F.Cu at (109.9, 76.2)
- added C30: 2.2uF/6.3V, Capacitor_SMD:C_0603_1608Metric, F.Cu at (113.4, 74.5)
- added C31: 0.1uF/16V, Capacitor_SMD:C_0402_1005Metric, F.Cu at (109.9, 78.2)
- added D1: SS54F-HF, SamacSys_Parts:SODFL4626X120N, F.Cu at (118.1, 88.5)
- added D2: SMBJ28CA-Q, SamacSys_Parts:DIONM5436X244N, F.Cu at (118.7, 84.2)
- added D3: B5819WS, SamacSys_Parts:SOD2613X100N, F.Cu at (117.2, 91.7)
- added IC1: TB67H450FNG,EL, SamacSys_Parts:SOIC127P600X175-9N, F.Cu at (138.6, 49.9)
- added IC2: TB67H450FNG,EL, SamacSys_Parts:SOIC127P600X175-9N, F.Cu at (138.6, 55.9)
- added JP1: SolderJumper_2_Open, Jumper:SolderJumper-2_P1.3mm_Open_RoundedPad1.0x1.5mm, F.Cu at (110.7, 88.2)
- added PS1: TPS563201DDCT, SamacSys_Parts:SOT95P280X110-6N, F.Cu at (124.9, 84.0)
- added R20: 4.7K/0.063w, Resistor_SMD:R_0402_1005Metric, F.Cu at (131.1, 47.7)
- added R21: 4.7K/0.063w, Resistor_SMD:R_0402_1005Metric, F.Cu at (131.1, 49.7)
- added R22: 4.7K/0.063w, Resistor_SMD:R_0402_1005Metric, F.Cu at (131.1, 51.7)
- added R23: 4.7K/0.063w, Resistor_SMD:R_0402_1005Metric, F.Cu at (131.1, 53.7)
- added R24: 4.7K/0.063w, Resistor_SMD:R_0402_1005Metric, F.Cu at (131.1, 55.7)
- added R25: 4.7K/0.063w, Resistor_SMD:R_0402_1005Metric, F.Cu at (131.1, 57.6)
- added R26: 4.7K/0.063w, Resistor_SMD:R_0402_1005Metric, F.Cu at (131.1, 59.6)
- added SW1: SW_Push, mylib:TSB008A2530A, F.Cu at (111.2, 100.0)
- added U2: STM32F103CBTx, Package_QFP:LQFP-48_7x7mm_P0.5mm, F.Cu at (137.2, 75.8)
- added U3: SN65HVD232, Package_SO:SOIC-8_3.9x4.9mm_P1.27mm, F.Cu at (104.3, 89.7)
- added U4: MT6816CT, Package_SO:SO-8_3.9x4.9mm_P1.27mm, F.Cu at (104.3, 76.6)
- added U6: ESP32-C3-WROOM-02, RF_Module:ESP32-C3-WROOM-02, F.Cu at (111.3, 57.9)
- U1: value STM32F103RBTx -> TPS54202DDC; footprint Package_QFP:LQFP-64_10x10mm_P0.5mm -> Package_TO_SOT_SMD:SOT-23-6
- moved U1 67.7 mm to (123.9, 89.0)
Connections:
- U1 pad 1: unconnected-(U1-VBAT-Pad1) -> GND
- U1 pad 2: unconnected-(U1-PC13-Pad2) -> Net-(U1-SW)
- U1 pad 3: unconnected-(U1-PC14-Pad3) -> Net-(U1-VIN)
- U1 pad 4: unconnected-(U1-PC15-Pad4) -> Net-(U1-FB)
- U1 pad 5: unconnected-(U1-PD0-Pad5) -> Net-(U1-EN)
- U1 pad 6: unconnected-(U1-PD1-Pad6) -> Net-(U1-BOOT)

Commit message: 작은 변경
Parts:
- added C28: 0.1uF/16V, Capacitor_SMD:C_0402_1005Metric, F.Cu at (75.2, 107.8)
- added C31: 0.1uF/16V, Capacitor_SMD:C_0402_1005Metric, F.Cu at (75.2, 109.7)
- added R21: 10K/0.063w, Resistor_SMD:R_0402_1005Metric, F.Cu at (72.3, 98.7)
- added R22: 4.7K/0.063w, Resistor_SMD:R_0402_1005Metric, F.Cu at (72.3, 100.7)
- added R23: NC_0R/0.1w, Resistor_SMD:R_0402_1005Metric, F.Cu at (72.3, 102.7)
- added R24: NC_0R/0.1w, Resistor_SMD:R_0402_1005Metric, F.Cu at (72.3, 104.7)
- added R27: 4.7K/0.063w, Resistor_SMD:R_0402_1005Metric, F.Cu at (72.3, 106.6)
- added R28: 10K/0.063w, Resistor_SMD:R_0402_1005Metric, F.Cu at (72.3, 108.6)
- added SW2: SW_Push, mylib:TSB008A2530A, F.Cu at (76.2, 115.0)
- added SW3: SW_Push, mylib:TSB008A2530A, F.Cu at (79.1, 100.0)
- added SW4: SW_Push, mylib:TSB008A2530A, F.Cu at (79.1, 104.5)
Connections:
- net ESP32_SPI2_MISO renamed FSPIQ
- net ESP32_SPI2_MOSI renamed FSPID
- net ESP32_SPI2_NSS renamed FSPICSO
- net ESP32_SPI2_SCK renamed FSPICLK
- net FSPIHD renamed Net-(LED3-K)
- net FSPIWP renamed Net-(LED2-K)
- U6 pad 11: Net-(J6-Pin_1) -> ESP_RX0
- U6 pad 12: Net-(J6-Pin_2) -> ESP_TX0
- U6 pad 15: GND -> ACT_BTN
- U6 pad 2: Net-(U6-EN) -> EN_BTN
- U6 pad 7: Net-(LED3-K) (its old number) -> unconnected-(U6-IO8-Pad7)
- U6 pad 8: Net-(LED2-K) (its old number) -> BOOT_BTN

Commit message: 회로도 대충 완성
Parts:
- added C15: 0.1uF/16V, Capacitor_SMD:C_0402_1005Metric, F.Cu at (148.6, 102.4)
- added C19: 0.1uF/16V, Capacitor_SMD:C_0402_1005Metric, F.Cu at (148.6, 104.3)
- added D2: SMBJ28CAQ-13-F, SamacSys_Parts:DIONM5336X250N, F.Cu at (143.9, 121.3)
- added D3: B5819WS, Diode_SMD:D_SOD-323, F.Cu at (149.9, 120.4)
- added D4: PRTR5V0U2X, Package_TO_SOT_SMD:SOT-143, F.Cu at (156.2, 122.9)
- added D5: SS54, PCM_Diode_SMD_AKL:D_SMC, F.Cu at (145.7, 114.5)
- added J3: USB_C, Connector_USB:USB_C_Receptacle_HRO_TYPE-C-31-M-12, F.Cu at (159.9, 115.8)
- added JP2: SolderJumper_3_Bridged123, Jumper:SolderJumper-3_P1.3mm_Bridged123_RoundedPad1.0x1.5mm, F.Cu at (165.5, 57.4)
- added JP3: SolderJumper_3_Bridged123, Jumper:SolderJumper-3_P1.3mm_Bridged123_RoundedPad1.0x1.5mm, F.Cu at (165.5, 61.2)
- added JP4: SolderJumper_3_Bridged123, Jumper:SolderJumper-3_P1.3mm_Bridged123_RoundedPad1.0x1.5mm, F.Cu at (165.5, 65.1)
- added JP5: SolderJumper_3_Bridged123, Jumper:SolderJumper-3_P1.3mm_Bridged123_RoundedPad1.0x1.5mm, F.Cu at (165.5, 68.9)
- added LED1: LED_0603_Red_WIFI, PCM_LED_SMD_AKL:LED_0603_1608Metric, F.Cu at (145.1, 103.1)
- added LED2: LED_0603_Blue_BLE, PCM_LED_SMD_AKL:LED_0603_1608Metric, F.Cu at (145.1, 106.4)
- added LED3: LED_0603_Green_PWR, PCM_LED_SMD_AKL:LED_0603_1608Metric, F.Cu at (158.2, 93.7)
- added LED4: LED_0603_Red_WIFI, PCM_LED_SMD_AKL:LED_0603_1608Metric, F.Cu at (158.2, 97.0)
- added LED5: LED_0603_Blue_BLE, PCM_LED_SMD_AKL:LED_0603_1608Metric, F.Cu at (158.2, 100.3)
- added R1: 511k/0.063w, Resistor_SMD:R_0402_1005Metric, F.Cu at (138.6, 111.0)
- added R10: 10k/0.063w, Resistor_SMD:R_0402_1005Metric, F.Cu at (138.6, 95.0)
- added R11: 10K/0.063w, Resistor_SMD:R_0402_1005Metric, F.Cu at (138.6, 97.0)
- added R12: 4.7K/0.063w, Resistor_SMD:R_0402_1005Metric, F.Cu at (138.6, 99.0)
- added R13: 10K/0.063w, Resistor_SMD:R_0402_1005Metric, F.Cu at (138.6, 101.0)
- added R14: 10k/0.063w, Resistor_SMD:R_0402_1005Metric, F.Cu at (138.6, 102.9)
- added R15: 10k/0.063w, Resistor_SMD:R_0402_1005Metric, F.Cu at (141.6, 93.0)
- added R16: 0R/0.063w, Resistor_SMD:R_0402_1005Metric, F.Cu at (141.6, 95.0)
- added R17: 0R/0.063w, Resistor_SMD:R_0402_1005Metric, F.Cu at (141.6, 97.0)
- added R18: 1k/0.063w, Resistor_SMD:R_0402_1005Metric, F.Cu at (172.1, 111.0)
- added R19: 1k/0.063w, Resistor_SMD:R_0402_1005Metric, F.Cu at (172.1, 113.0)
- added R2: 105k/0.063w, Resistor_SMD:R_0402_1005Metric, F.Cu at (138.6, 113.0)
- added R21: 1k/0.063w, Resistor_SMD:R_0402_1005Metric, F.Cu at (172.1, 115.0)
- added R22: 1k/0.063w, Resistor_SMD:R_0402_1005Metric, F.Cu at (172.1, 117.0)
- added R24: NC_4.7K, Resistor_SMD:R_0402_1005Metric, F.Cu at (167.2, 111.0)
- added R25: 4.7K, Resistor_SMD:R_0402_1005Metric, F.Cu at (167.2, 113.0)
- added R3: 10k/0.063w, Resistor_SMD:R_0402_1005Metric, F.Cu at (138.6, 115.0)
- added R37: 4.7K/0.063w, Resistor_SMD:R_0402_1005Metric, F.Cu at (141.6, 99.0)
- added R38: 4.7K/0.063w, Resistor_SMD:R_0402_1005Metric, F.Cu at (141.6, 101.0)
- added R39: 4.7k/0.063w, Resistor_SMD:R_0402_1005Metric, F.Cu at (167.2, 115.0)
- added R4: 33.2k/0.063w, Resistor_SMD:R_0402_1005Metric, F.Cu at (138.6, 117.0)
- added R5: 10k/0.063w, Resistor_SMD:R_0402_1005Metric, F.Cu at (138.6, 119.0)
- added R6: 49.9R/0.063w, Resistor_SMD:R_0402_1005Metric, F.Cu at (138.6, 121.0)
- added R7: 100k/0.063w, Resistor_SMD:R_0402_1005Metric, F.Cu at (138.6, 123.0)
- added R8: 13.3k/0.063w, Resistor_SMD:R_0402_1005Metric, F.Cu at (138.6, 125.0)
- added R9: 4.7K/0.063w, Resistor_SMD:R_0402_1005Metric, F.Cu at (138.6, 93.0)
- added RT1: NCP18XH103F03RB, SamacSys_Parts:THRMC1608X95N, F.Cu at (151.7, 102.4)
- added S1: TSB008A2518A, SamacSys_Parts:TSB008A2518A, F.Cu at (148.9, 94.3)
- added S2: TSB008A2518A, SamacSys_Parts:TSB008A2518A, F.Cu at (148.9, 99.0)
- added S3: TSB008A2518A, SamacSys_Parts:TSB008A2518A, F.Cu at (166.1, 94.3)
- added S4: TSB008A2518A, SamacSys_Parts:TSB008A2518A, F.Cu at (166.1, 99.0)
- added U4: TL431AIDBZR, SamacSys_Parts:SOT95P237X112-3N, F.Cu at (162.5, 103.5)
- H1, H2, H3, H4: value MountingHole_M3 -> MountingHole
- U2: moved to B.Cu
- moved U6 18.6 mm to (106.1, 40.1)
- moved U2 6.51 mm to (132.4, 71.5), turned to 180 degrees
- renumbered C31 to C29, C28 to C31, C29 to C32, C30 to C33, R20 to R27, R25 to R28, R28 to R30, R26 to R31, R21 to R32, R27 to R33, R22 to R34, R23 to R35, R24 to R36, U4 to U5
Connections:
- R35 pad 1: D- -> USB_DM
- R36 pad 1: D+ -> USB_DP
- U2 pad 10: unconnected-(U2-PA0-Pad10) -> ADC_VREF_2V5
- U2 pad 11: unconnected-(U2-PA1-Pad11) -> TEMP
- U2 pad 12: unconnected-(U2-PA2-Pad12) -> ESP32_UART_RX
- U2 pad 13: unconnected-(U2-PA3-Pad13) -> ESP32_UART_TX
- U2 pad 14: unconnected-(U2-PA4-Pad14) -> ADC_ENC
- U2 pad 15: unconnected-(U2-PA5-Pad15) -> SPI1_CLK
- U2 pad 16: unconnected-(U2-PA6-Pad16) -> SPI1_MISO
- U2 pad 17: unconnected-(U2-PA7-Pad17) -> SPI1_MOSI
- U2 pad 18: unconnected-(U2-PB0-Pad18) -> MT6816_CSN
- U2 pad 21: unconnected-(U2-PB10-Pad21) -> WS2812_SIGNAL
- U2 pad 25: unconnected-(U2-PB12-Pad25) -> IN_B-
- U2 pad 26: unconnected-(U2-PB13-Pad26) -> IN_B+
- U2 pad 27: unconnected-(U2-PB14-Pad27) -> IN_A-
- U2 pad 28: unconnected-(U2-PB15-Pad28) -> IN_A+
- U2 pad 29: unconnected-(U2-PA8-Pad29) -> VREF_PWM_A
- U2 pad 30: unconnected-(U2-PA9-Pad30) -> VREF_PWM_B
- U2 pad 32: unconnected-(U2-PA11-Pad32) -> Net-(U2-PA11)
- U2 pad 33: unconnected-(U2-PA12-Pad33) -> Net-(U2-PA12)
- U2 pad 34: unconnected-(U2-PA13-Pad34) -> SWDIO
- U2 pad 37: unconnected-(U2-PA14-Pad37) -> SWCLK
- U2 pad 38: unconnected-(U2-PA15-Pad38) -> LED1
- U2 pad 39: unconnected-(U2-PB3-Pad39) -> LED2
- U2 pad 40: unconnected-(U2-PB4-Pad40) -> BTN1
- U2 pad 41: unconnected-(U2-PB5-Pad41) -> BTN2
- U2 pad 42: unconnected-(U2-PB6-Pad42) -> UART1_TX
- U2 pad 43: unconnected-(U2-PB7-Pad43) -> UART1_RX
- U2 pad 45: unconnected-(U2-PB8-Pad45) -> CAN_RX
- U2 pad 46: unconnected-(U2-PB9-Pad46) -> CAN_TX
- U6 pad 10: FSPICSO -> unconnected-(U6-IO10-Pad10)
- U6 pad 16: FSPIQ -> unconnected-(U6-IO2-Pad16)
- U6 pad 5: FSPICLK -> unconnected-(U6-IO6-Pad5)
- U6 pad 6: FSPID -> unconnected-(U6-IO7-Pad6)
Other:
- copper layers 2 -> 4

Commit message: 수정
Parts:
- removed SW1, SW2, SW3, SW4: SW_Push, mylib:TSB008A2530A
- added C1: 22uF/10V, Capacitor_SMD:C_1206_3216Metric, F.Cu at (91.2, 113.7)
- added C10: CL31A106KBHNNNE, Capacitor_SMD:C_1206_3216Metric, F.Cu at (91.2, 133.8)
- added C11: 22uF/10V, Capacitor_SMD:C_1206_3216Metric, F.Cu at (91.2, 137.1)
- added C12: 22uF/10V, Capacitor_SMD:C_1206_3216Metric, F.Cu at (91.2, 140.5)
- added C13: 75pF/50V, Capacitor_SMD:C_0402_1005Metric, F.Cu at (95.5, 118.9)
- added C14: 0.1uF/50V, Capacitor_SMD:C_0402_1005Metric, F.Cu at (104.4, 137.8)
- added C16: 4.7uF/10V, Capacitor_SMD:C_0603_1608Metric, F.Cu at (107.9, 138.1)
- added C17: 0.1uF/50V, Capacitor_SMD:C_0402_1005Metric, F.Cu at (104.4, 139.8)
- added C18: 0.1uF/50V, Capacitor_SMD:C_0402_1005Metric, F.Cu at (104.4, 141.8)
- added C2: CL31A106KBHNNNE, Capacitor_SMD:C_1206_3216Metric, F.Cu at (91.2, 117.0)
- added C20: 0.1uF/50V, Capacitor_SMD:C_0402_1005Metric, F.Cu at (104.4, 143.7)
- added C21: 0.1uF/50V, Capacitor_SMD:C_0402_1005Metric, F.Cu at (104.4, 145.7)
- added C22: 12pF/50V, Capacitor_SMD:C_0402_1005Metric, F.Cu at (104.4, 147.7)
- added C23: 12pF/50V, Capacitor_SMD:C_0402_1005Metric, F.Cu at (104.4, 149.6)
- added C24: 0.1uF/50V, Capacitor_SMD:C_0402_1005Metric, F.Cu at (123.9, 137.8)
- added C25: 0.1uF/50V, Capacitor_SMD:C_0402_1005Metric, F.Cu at (123.9, 139.8)
- added C26: 0.1uF/50V, Capacitor_SMD:C_0402_1005Metric, F.Cu at (123.9, 141.8)
- added C27: 0.1uF/50V, Capacitor_SMD:C_0402_1005Metric, F.Cu at (123.9, 143.7)
- added C28: 10uF/6.3V, Capacitor_SMD:C_0603_1608Metric, F.Cu at (118.5, 138.1)
- added C3: 22uF/10V, Capacitor_SMD:C_1206_3216Metric, F.Cu at (91.2, 120.4)
- added C30: 0.1uF/50V, Capacitor_SMD:C_0402_1005Metric, F.Cu at (117.9, 142.8)
- added C34: 10uF/16V, Capacitor_SMD:C_0805_2012Metric, F.Cu at (96.3, 130.5)
- added C35: 10uF/16V, Capacitor_SMD:C_0805_2012Metric, F.Cu at (96.3, 133.5)
- added C36: 0.1uF/50V, Capacitor_SMD:C_0402_1005Metric, F.Cu at (95.5, 120.9)
- added C4: 0.1uF/50V, Capacitor_SMD:C_0402_1005Metric, F.Cu at (95.5, 113.0)
- added C5: 0.1uF/50V, Capacitor_SMD:C_0402_1005Metric, F.Cu at (95.5, 115.0)
- added C6: CL31A106KBHNNNE, Capacitor_SMD:C_1206_3216Metric, F.Cu at (91.2, 123.7)
- added C7: CL31A106KBHNNNE, Capacitor_SMD:C_1206_3216Metric, F.Cu at (91.2, 127.1)
- added C8: CL31A106KBHNNNE, Capacitor_SMD:C_1206_3216Metric, F.Cu at (91.2, 130.4)
- added C9: 0.1uF/50V, Capacitor_SMD:C_0402_1005Metric, F.Cu at (95.5, 116.9)
- added J1: PC_CONN, Connector_JST:JST_SH_SM05B-SRSS-TB_1x05-1MP_P1.00mm_Horizontal, F.Cu at (116.0, 105.0)
- added J10: VBUS_EN, Connector_PinHeader_2.54mm:PinHeader_1x02_P2.54mm_Vertical, F.Cu at (124.4, 110.1)
- added J2: MT6816_CONN, Connector_JST:JST_SH_SM05B-SRSS-TB_1x05-1MP_P1.00mm_Horizontal, F.Cu at (115.8, 123.4)
- added J4: DEBUG, Connector_JST:JST_SH_SM03B-SRSS-TB_1x03-1MP_P1.00mm_Horizontal, F.Cu at (106.8, 105.3)
- added J5: CAN_IN, Connector_JST:JST_SH_SM06B-SRSS-TB_1x06-1MP_P1.00mm_Horizontal, F.Cu at (70.7, 53.4)
- added J6: CAN_OUT, Connector_JST:JST_SH_SM06B-SRSS-TB_1x06-1MP_P1.00mm_Horizontal, F.Cu at (71.4, 86.7)
- added J7: ESP_DOWNLOAD, Connector_JST:JST_SH_SM03B-SRSS-TB_1x03-1MP_P1.00mm_Horizontal, F.Cu at (106.9, 123.4)
- added J8: BOOT_EN, Connector_PinHeader_2.54mm:PinHeader_1x02_P2.54mm_Vertical, F.Cu at (109.3, 112.3)
- added J9: WS2812_OUT, Connector_JST:JST_SH_SM03B-SRSS-TB_1x03-1MP_P1.00mm_Horizontal, F.Cu at (106.9, 131.0)
- added L1: 2.2uH, Inductor_SMD:L_Sunlord_SWPA252012S, F.Cu at (99.0, 113.8)
- added L2: 15uH, Inductor_SMD:L_Sunlord_SWPA4020S, F.Cu at (96.9, 137.8)
- added R20: 0.1/0.25w, Resistor_SMD:R_1206_3216Metric, F.Cu at (128.1, 138.5)
- added R23: 0.1/0.25w, Resistor_SMD:R_1206_3216Metric, F.Cu at (128.1, 141.8)
- added R26: 120/0.1w, Resistor_SMD:R_0603_1608Metric, F.Cu at (122.7, 128.5)
- added R29: 120/0.1w, Resistor_SMD:R_0603_1608Metric, F.Cu at (118.5, 140.6)
- added U7: TPS563203, Package_TO_SOT_SMD:SOT-563, F.Cu at (99.1, 117.1)
- JP1: value SolderJumper_2_Open -> CAN_END_PAD
- JP2: value SolderJumper_3_Bridged123 -> PAD_OUTA_P
- JP3: value SolderJumper_3_Bridged123 -> PAD_OUTA_M
- JP4: value SolderJumper_3_Bridged123 -> PAD_OUTB_P
- JP5: value SolderJumper_3_Bridged123 -> PAD_OUTB_M
- R3: value 10k/0.063w -> 100k/0.063w
- R4: value 33.2k/0.063w -> 135k/0.063w
- R5: value 10k/0.063w -> 30k/0.063w
- U3, U5: moved to B.Cu
- moved J3 66.3 mm to (94.9, 102.9)
- moved U3 40.8 mm to (144.4, 82.2), turned to 180 degrees
- moved U5 12.9 mm to (111.0, 65.6), turned to 180 degrees
- moved JP3 12.2 mm to (153.5, 63.6)
- moved JP4 12.2 mm to (153.5, 67.4)
- moved JP2 12.2 mm to (153.5, 59.8)
- moved JP5 12.2 mm to (153.5, 71.3)
- moved C29 9.58 mm to (74.0, 100.2)
- moved JP1 9.57 mm to (103.7, 94.7)
- moved R30 8.47 mm to (71.1, 100.2)
- moved U6 7.60 mm to (106.0, 32.5)
- moved C31 5.70 mm to (74.0, 102.2)
- moved R34 5.69 mm to (71.1, 106.2)
- moved R35 5.69 mm to (71.1, 108.2)
- moved R36 5.69 mm to (71.1, 110.2)
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Connections:
- R3 pad 1: Net-(PS1-EN) -> 5V
- R3 pad 2: 5V -> Net-(U7-EN)
- R4 pad 2: Net-(PS1-VFB) -> Net-(U7-FB)
- R5 pad 1: Net-(PS1-VFB) -> Net-(U7-FB)

Commit message: 3V3 LDO변경 및 대략적 위치 세팅
Parts:
- removed the C28 at (109.9, 74.2)
- removed C35: 10uF/16V, Capacitor_SMD:C_0805_2012Metric
- removed C36: 0.1uF/50V, Capacitor_SMD:C_0402_1005Metric
- removed D1: SS54F-HF, SamacSys_Parts:SODFL4626X120N
- removed the D2 at (143.9, 121.3)
- removed the D2 at (118.7, 84.2)
- removed the D3 at (149.9, 120.4)
- removed the D3 at (117.2, 91.7)
- removed D5: SS54, PCM_Diode_SMD_AKL:D_SMC
- removed J10: VBUS_EN, Connector_PinHeader_2.54mm:PinHeader_1x02_P2.54mm_Vertical
- removed J3: USB_C, Connector_USB:USB_C_Receptacle_HRO_TYPE-C-31-M-12
- removed JP2: PAD_OUTA_P, Jumper:SolderJumper-3_P1.3mm_Bridged123_RoundedPad1.0x1.5mm
- removed JP3: PAD_OUTA_M, Jumper:SolderJumper-3_P1.3mm_Bridged123_RoundedPad1.0x1.5mm
- removed JP4: PAD_OUTB_P, Jumper:SolderJumper-3_P1.3mm_Bridged123_RoundedPad1.0x1.5mm
- removed JP5: PAD_OUTB_M, Jumper:SolderJumper-3_P1.3mm_Bridged123_RoundedPad1.0x1.5mm
- removed L1: 2.2uH, Inductor_SMD:L_Sunlord_SWPA252012S
- removed R16, R17: 0R/0.063w, Resistor_SMD:R_0402_1005Metric
- removed R24: NC_4.7K, Resistor_SMD:R_0402_1005Metric
- removed R24: 4.7K/0.063w, Resistor_SMD:R_0402_1005Metric
- removed R25: 4.7K, Resistor_SMD:R_0402_1005Metric
- removed R3: 100k/0.063w, Resistor_SMD:R_0402_1005Metric
- removed R35, R36: NC_0R/0.1w, Resistor_SMD:R_0402_1005Metric
- removed R4: 135k/0.063w, Resistor_SMD:R_0402_1005Metric
- removed R5: 30k/0.063w, Resistor_SMD:R_0402_1005Metric
- removed U7: TPS563203, Package_TO_SOT_SMD:SOT-563
- added D2: SMBJ28CAQ-13-F, SamacSys_Parts:DIONM5336X250N, F.Cu at (79.6, 43.3)
- added D3: B5819WS, Diode_SMD:D_SOD-323, F.Cu at (72.4, 143.7)
- added IC3: TLV74033PDBVR, SamacSys_Parts:SOT95P280X145-5N, F.Cu at (30.4, 109.2)
- added TP1: PAD_4_15, New_Footprints:custom_pad_4_15, B.Cu at (187.8, 75.8)
- added TP2: PAD_4_15, New_Footprints:custom_pad_4_15, B.Cu at (180.9, 76.7)
- added TP3: PAD_4_15, New_Footprints:custom_pad_4_15, B.Cu at (175.9, 76.7)
- added TP4: PAD_4_15, New_Footprints:custom_pad_4_15, B.Cu at (170.9, 76.7)
- added Y1: YSX321SL_12Mhz, Crystal:Crystal_SMD_3225-4Pin_3.2x2.5mm, B.Cu at (351.5, 48.8)
- C1: value 22uF/10V -> 0.1uF/50V; footprint Capacitor_SMD:C_1206_3216Metric -> Capacitor_SMD:C_0402_1005Metric
- C14, C16, C17, C18, C20, C21, C22, C23, C24, C25, C26, C27, C28, C30, IC1, IC2, R10, R14, R15, R18, R19, R21 (x2), R22 (x2), R37, R38, RT1, U6: moved to B.Cu
- C3: value 22uF/10V -> 1uF/10V; footprint Capacitor_SMD:C_1206_3216Metric -> Capacitor_SMD:C_0402_1005Metric
- C34: value 10uF/16V -> 10uF/6.3V; footprint Capacitor_SMD:C_0805_2012Metric -> Capacitor_SMD:C_0603_1608Metric
- C5: value 0.1uF/50V -> 1uF/10V
- D4: value PRTR5V0U2X -> SS54; footprint Package_TO_SOT_SMD:SOT-143 -> SamacSys_Parts:DIOM5126X245N
- moved C21 256.6 mm to (360.1, 124.5), turned to 180 degrees
- moved C22 249.1 mm to (343.8, 78.9), turned to 180 degrees
- moved C23 249.1 mm to (343.8, 80.8), turned to 180 degrees
- moved C17 219.3 mm to (320.4, 101.7), turned to 180 degrees
- moved C18 219.3 mm to (320.4, 103.7), turned to 180 degrees
- moved C20 219.3 mm to (320.4, 105.6), turned to 180 degrees
- moved R37 217.8 mm to (355.6, 58.4), turned to 180 degrees
- moved R38 216.8 mm to (354.8, 61.6), turned to 180 degrees
- moved C16 212.6 mm to (317.0, 100.0), turned to 180 degrees
- moved RT1 211.9 mm to (360.0, 63.2), turned to 180 degrees
- moved C14 209.6 mm to (310.3, 99.0), turned to 180 degrees
- moved R10 209.0 mm to (343.7, 54.4), turned to 180 degrees
- moved U2 208.9 mm to (337.9, 34.1)
- moved R14 188.5 mm to (325.9, 81.8), turned to 180 degrees
- moved R15 182.7 mm to (323.0, 71.8), turned to 180 degrees
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Connections:
- C3 pad 1: 3V3 -> 5V
- C34 pad 1: 5V -> 3V3
- C5 pad 1: Net-(U7-BST) -> 3V3
- C5 pad 2: Net-(U7-SW) -> GND
- D4 pad 1: GND -> VCC
- D4 pad 2: USB_DP -> VCC_IN
- U2 pad 32: Net-(U2-PA11) -> unconnected-(U2-PA11-Pad32)
- U2 pad 33: Net-(U2-PA12) -> unconnected-(U2-PA12-Pad33)
- U6 pad 13: Net-(U6-IO18) -> unconnected-(U6-IO18-Pad13)
- U6 pad 14: Net-(U6-IO19) -> unconnected-(U6-IO19-Pad14)
Routing:
- net 5V: track 0.00 -> 5.40 mm
- net 3V3: track 0.00 -> 3.93 mm

Commit message: 중간 저장
Parts:
- removed C29: 0.1uF/16V, Capacitor_SMD:C_0402_1005Metric
- removed the C31 at (109.9, 78.2)
- removed the C31 at (103.5, 103.5)
- removed PS1: TPS563201DDCT, SamacSys_Parts:SOT95P280X110-6N
- removed the R21 at (183.8, 47.6)
- removed the R21 at (178.5, 56.3)
- removed the R22 at (183.8, 49.6)
- removed the R22 at (178.5, 58.3)
- removed R30: 10K/0.063w, Resistor_SMD:R_0402_1005Metric
- removed R37, R38: 4.7K/0.063w, Resistor_SMD:R_0402_1005Metric
- removed S4: TSB008A2518A, SamacSys_Parts:TSB008A2518A
- added C31: 0.1uF/16V, Capacitor_SMD:C_0402_1005Metric, F.Cu at (79.8, 74.6)
- added C35: 0.1uF/50V, Capacitor_SMD:C_0402_1005Metric, B.Cu at (61.5, 86.2)
- added C36: 1uF/10V, Capacitor_SMD:C_0402_1005Metric, B.Cu at (61.5, 87.2)
- added R21: 1k/0.063w, Resistor_SMD:R_0402_1005Metric, B.Cu at (63.0, 65.2)
- added R22: 1k/0.063w, Resistor_SMD:R_0402_1005Metric, B.Cu at (65.5, 65.7)
- C32, C33, R20, R23, R29, R33, R34, U4: moved to B.Cu
- TP1, TP2, TP3, TP4: value PAD_4_15 -> PAD_4_12; footprint New_Footprints:custom_pad_4_15 -> New_Footprints:custom_pad_2_5
- U3: moved to F.Cu
- moved C21 301.2 mm to (61.5, 85.2)
- moved C16 298.7 mm to (18.8, 83.0), turned to 90 degrees
- moved RT1 293.4 mm to (67.0, 77.8), turned to 90 degrees
- moved Y1 290.6 mm to (62.8, 82.4)
- moved C23 282.3 mm to (61.5, 80.1), turned to 0 degrees
- moved C22 280.3 mm to (63.5, 80.1), turned to 0 degrees
- moved U2 279.8 mm to (61.0, 73.9), turned to 90 degrees
- moved R10 277.4 mm to (67.5, 80.4), turned to 90 degrees
- moved C17 265.8 mm to (56.6, 69.7), turned to 90 degrees
- moved R14 262.5 mm to (63.5, 85.2), turned to 0 degrees
- moved C18 257.6 mm to (65.1, 69.6), turned to 0 degrees
- moved C20 256.6 mm to (65.3, 78.1), turned to -90 degrees
- moved R15 256.4 mm to (66.7, 75.2), turned to -90 degrees
- moved C14 244.6 mm to (66.5, 80.3), turned to -90 degrees
- moved R9 213.7 mm to (26.7, 65.7), turned to -90 degrees
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Connections:
- TP1 pad 1: OUT_A+ -> OUT_A-
- TP2 pad 1: OUT_A- -> OUT_A+
- TP3 pad 1: OUT_B+ -> OUT_B-
- TP4 pad 1: OUT_B- -> OUT_B+
- U6 pad 15: ACT_BTN -> unconnected-(U6-IO3-Pad15)
Routing:
- net ESP32_UART_RX: track 0.00 -> 51.3 mm, vias 0 -> 2
- net ESP32_UART_TX: track 0.00 -> 49.0 mm, vias 0 -> 2
- net WS2812_SIGNAL: track 0.00 -> 40.1 mm, vias 0 -> 1
- net IN_A-: track 0.00 -> 21.3 mm, vias 0 -> 2
- net IN_A+: track 0.00 -> 19.8 mm, vias 0 -> 2
- net MT6816_CSN: track 0.00 -> 19.3 mm, vias 0 -> 2
- net ADC_VREF_2V5: track 0.00 -> 17.7 mm
- net IN_B-: track 0.00 -> 16.3 mm, vias 0 -> 2
- net IN_B+: track 0.00 -> 14.6 mm, vias 0 -> 2
- net EN_BTN: track 0.00 -> 14.3 mm, vias 0 -> 1
- net SPI1_CLK: track 0.00 -> 14.3 mm, vias 0 -> 2
- net SPI1_MISO: track 0.00 -> 13.5 mm, vias 0 -> 2
- net CAN_H: track 0.00 -> 13.3 mm, vias 0 -> 1
- net SPI1_MOSI: track 0.00 -> 12.8 mm, vias 0 -> 2
- net TEMP: track 0.00 -> 12.3 mm, vias 0 -> 2
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