File: 1.hardware/motor_42/motor_42.kicad_pcb (KiCad board)
At the start: 4 copper layers, 40 x 40 mm, 103 parts, among them IC1 TB67H450FNG,EL, IC2 TB67H450FNG,EL, IC3 TLV74033PDBVR, J1 PC_CONN, J2 MT6816_CONN, J4 DEBUG, J5 CAN_IN, J6 CAN_OUT, J7 ESP_DOWNLOAD, J8 BOOT_EN, J9 WS2812_OUT, U1 TPS54202DDC, U2 STM32F103CBTx, U3 SN65HVD232, U4 TL431AIDBZR, U5 MT6816CT, U6 ESP32-C3-WROOM-02, Y1 YSX321SL_12Mhz

Commit message: 얼추 다 그림
Parts:
- removed C1: 0.1uF/50V, Capacitor_SMD:C_0402_1005Metric
- removed C3, C5: 1uF/10V, Capacitor_SMD:C_0402_1005Metric
- removed C34: 10uF/6.3V, Capacitor_SMD:C_0603_1608Metric
- removed IC3: TLV74033PDBVR, SamacSys_Parts:SOT95P280X145-5N
- removed J9: WS2812_OUT, Connector_JST:JST_SH_SM03B-SRSS-TB_1x03-1MP_P1.00mm_Horizontal
- removed LED3: LED_0603_Green_PWR, PCM_LED_SMD_AKL:LED_0603_1608Metric
- removed the R23 at (83.7, 105.4)
- removed R27: 4.7K/0.063w, Resistor_SMD:R_0402_1005Metric
- removed R39: 4.7k/0.063w, Resistor_SMD:R_0402_1005Metric
- L2: value 15uH -> 10uH
- moved C15 71.2 mm to (68.1, 71.5), turned to 90 degrees
- moved C19 71.1 mm to (74.5, 71.5), turned to 90 degrees
- moved R13 66.1 mm to (71.9, 71.5), turned to -90 degrees
- moved R11 64.5 mm to (70.7, 71.5), turned to -90 degrees
- moved R8 52.6 mm to (76.2, 69.1), turned to 90 degrees
- moved C13 52.3 mm to (76.2, 72.1)
- moved R6 52.3 mm to (77.2, 72.1)
- moved R7 52.3 mm to (77.2, 70.2)
- moved U1 52.3 mm to (79.9, 70.9)
- moved C9 51.8 mm to (78.3, 73.4), turned to -90 degrees
- moved C4 51.7 mm to (81.5, 68.6)
- moved R1 51.7 mm to (79.6, 68.6)
- moved R2 51.7 mm to (77.7, 68.6)
- moved C2 51.7 mm to (79.1, 66.8)
- moved D3 51.6 mm to (80.5, 63.9)
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Connections:
- C11 pad 1: 5V -> 3V3
- C12 pad 1: 5V -> 3V3
- L2 pad 2: 5V -> 3V3
- R6 pad 1: 5V -> 3V3
- U2 pad 21: WS2812_SIGNAL -> unconnected-(U2-PB10-Pad21)
- U6 pad 3: Net-(LED5-K) -> unconnected-(U6-IO4-Pad3)
- U6 pad 4: Net-(LED4-K) -> unconnected-(U6-IO5-Pad4)
- U6 pad 6: unconnected-(U6-IO7-Pad6) -> Net-(LED5-K)
- U6 pad 7: unconnected-(U6-IO8-Pad7) -> Net-(LED4-K)
Routing:
- net 3V3: track 15.8 -> 75.0 mm, vias 0 -> 35
- net WS2812_SIGNAL: track 40.1 -> 0.00 mm, vias 1 -> 0
- net ESP_RX0: track 0.00 -> 39.6 mm, vias 0 -> 2
- net ESP_TX0: track 0.00 -> 37.6 mm, vias 0 -> 2
- net CAN_L: track 11.0 -> 47.1 mm, vias 1 -> 3
- net CAN_H: track 13.3 -> 48.3 mm, vias 1 -> 3
- net GND: track 0.00 -> 34.9 mm, vias 0 -> 79
- net SPI1_MISO: track 13.5 -> 36.3 mm, vias 2 -> 4
- net SPI1_MOSI: track 12.8 -> 35.5 mm, vias 2 -> 4
- net LED1: track 0.00 -> 22.5 mm, vias 0 -> 2
- net SPI1_CLK: track 14.3 -> 36.4 mm, vias 2 -> 4
- net LED2: track 0.00 -> 21.4 mm, vias 0 -> 2
- net CAN_TX: track 0.00 -> 18.9 mm, vias 0 -> 2
- net CAN_RX: track 0.00 -> 18.7 mm, vias 0 -> 2
- net BTN2: track 0.00 -> 11.9 mm, vias 0 -> 1
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- added copper zone on F.Cu, net 3V3
- added copper zone on In1.Cu, net 3V3
- added copper zone on B.Cu, net GND
- added copper zone on F.Cu, net GND
- added copper zone on In2.Cu, net GND
- added copper zone on B.Cu, net VCC
- added copper zone on F.Cu, net VCC
- added copper zone on In1.Cu, net VCC
- added copper zone on F.Cu, net VCC_IN
- added copper zone on In1.Cu, net VCC_IN

Commit message: 실크 업데이트
Other:
- board text added: "12Mhz"
- board text added: "24V MAX STEPPER MOTOR DRIVER"
- board text added: "A+A-"
- board text added: "ADC_ENC"
- board text added: "ADF_2V5"
- board text added: "B+B-"
- board text added: "BOOT0"
- board text added: "BTN1"
- board text added: "BTN2"
- board text added: "CAN_END"
- board text added: "CAN_H"
- board text added: "CAN_IN"
- board text added: "CAN_L"
- board text added: "CAN_OUT"
- board text added: "DRIVER"
- board text added: "ESP32C3"
- board text added: "ESP_DBG"
- board text added: "ESP_EN_BTN"
- board text added: "GND"
- board text added: "LED1"
- board text added: "LED2"
- board text added: "MT6816_CONN"
- board text added: "MT6816_MAGNETIC"
- board text added: "STM32F103"
- board text added: "STM_DBG"
- board text added: "STM_UART"
- board text added: "VCC_IN"
