File: 1.hardware/motor_42/Power.kicad_sch (KiCad schematic)
At the start: 24 parts, among them U1 TPS54202DDC

Commit message: 코드 추가
Parts:
- R5: value 13.3k/0.063w -> 22k/0.063w
Changed lines of the file:
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@@
 	(generator_version "9.0")
 	(paper "A")
+	(rectangle
+		(start 151.13 102.87)
+		(end 173.99 121.92)
+		(stroke
+			(width 0)
+			(type default)
+		)
+		(fill
+			(type none)
+		)
+	)
 	(text "5V"
 		(exclude_from_sim no)
@@
 			)
 		)
-		(property "Value" "13.3k/0.063w"
+		(property "Value" "22k/0.063w"
 			(at 158.75 111.7599 0)
 			(effects
